File: Boards/Avionics/HYDRA_V2/HYDRA_V2/HYDRA_V2.kicad_sch (KiCad schematic)
At the start: 17 parts, among them IC1 MAX31855KASA+T, IC2 MAX31855KASA+T, IC3 MAX31855KASA+T, Q1 IRLB3813PBF-ND, Q2 IRLB3813PBF-ND, Q3 IRLB3813PBF-ND, U1 MAX485_MODULE_5V_LOGIC_TLL_TO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

Commit message: Hydrav2
Parts:
- added C1, C2, C3: 0.1uF, symbol Device:C_Small
- added D4, D5, D6: LED, symbol Device:LED
- added J1, J2, J3, J4: 1723103102, 1723103102:CONN02_1723103102_MOL, symbol 1723103102:1723103102
- added J5, J6: 1723103103, 1723103103:MOLEX_1723103103, symbol 1723103103:1723103103
- added R6: 500, symbol Device:R
- added R7: 150, symbol Device:R
- added R8: 62, symbol Device:R
- added U3, U4, U5: ThermoConnector, ThermoPCBConnector:Thermo Type K PCB Connector, symbol ThermoPCBConnector:ThermoPCBConnector
- added U6, U7, U8: ~, symbol Mini Dc-Dc:MiniDCDCBoost
Connections:
- net +12V: now also D4.2 (A), J1.4 (SHIELD2), J2.4 (SHIELD2), J3.4 (SHIELD2), U6.3 (OUT+)
- net +3.3V: now also C1.2, C2.2, C3.2, D6.2 (A), U8.3 (OUT+)
- net +5V: now also D5.2 (A), U7.3 (OUT+)
- net GND: now also C1.1, C2.1, C3.1, J1.1, J1.2, J2.1, J2.2, J3.1, J3.2, J4.1, J4.2, J5.S1 (SHIELD1), J5.S2 (SHIELD2), R6.2, R7.2, R8.2, U6.2 (IN-), U6.4 (OUT-), U7.2 (IN-), U7.4 (OUT-), U8.2 (IN-), U8.4 (OUT-)
- net RS_A: now also J4.3 (SHIELD1)
- net RS_B: now also J4.4 (SHIELD2)
- net at D2.2 (A), Q2.2 (D): now also J2.3 (SHIELD1)
- net at D3.2 (A), Q3.2 (D): now also J3.3 (SHIELD1)
- net at D1.2 (A), Q1.2 (D): now also J1.3 (SHIELD1)
- removed net Thermocouple_CS: IC1.6 (~{CS}), IC2.6 (~{CS}), IC3.6 (~{CS})
- removed net Thermocouple_T+: IC1.3 (T+), IC2.3 (T+), IC3.3 (T+)
- removed net Thermocouple_T-: IC1.2 (T-), IC2.2 (T-), IC3.2 (T-)
- new net: D6.1 (K), R8.1
- new net: D4.1 (K), R6.1
- new net: D5.1 (K), R7.1
- new net Servo_GND: J5.3, J6.3
- new net Servo_PWM1: J6.2
- new net Servo_PWM2: J5.2
- new net Servo_VCC: J5.1, J6.1
- new net Thermocouple1_T+: IC1.3 (T+), U3.1 (T+)
- new net Thermocouple1_T-: IC1.2 (T-), U3.2 (T-)
- new net Thermocouple2_T+: IC2.3 (T+), U4.1 (T+)
- new net Thermocouple2_T-: IC2.2 (T-), U4.2 (T-)
- new net Thermocouple3_T+: IC3.3 (T+), U5.1 (T+)
- new net Thermocouple3_T-: IC3.2 (T-), U5.2 (T-)
- new net Thermocouple_CS1: IC1.6 (~{CS})
- new net Thermocouple_CS2: IC2.6 (~{CS})
- new net Thermocouple_CS3: IC3.6 (~{CS})
- new net VIN: U6.1 (IN+), U7.1 (IN+), U8.1 (IN+)
Other:
- note added: "DC-DC Converter"
- note added: "LED Driver"
- note added: "Power Requirements: 12.7V - 12Vx 12.7V - 8.4V 12.7V - 5Vx 5V - 3.3Vx"
- note added: "Requirements: 3x Solenoid Valves (Output)x 3x Thermopairs (Input) x 3x Pressure Transducers (Input) x 2x Servo Motors (Output)x"
- note added: "Vin = 12.7V"
- note removed: "Power Requirements: 12.7V - 12V 12.7V - 8.4V 12.7V - 5V 5V - 3.3V"
- note removed: "Requirements: 3x Solenoid Valves (Output) 3x Thermopairs (Input) x 3x Pressure Transducers (Input) x 2x Servo Motors (Output)"
- moved on the sheet: A1, D1, D2, D3, IC1, Q1, Q2, Q3, R1, R2, R3, R4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
